Commit message: Fixed mimic gazebo simulation; added mimic GUI simulation

File: urdf/left_open_manipulator.urdf.xacro (robot description, xacro)
@@ -7,5 +7,5 @@
   <xacro:include filename="$(find open_manipulator_description)/urdf/materials.xacro" />
   <!-- Import Transmission -->
-  <xacro:include filename="$(find open_manipulator_description)/urdf/transmission.xacro" />
+  <xacro:include filename="$(find open_manipulator_description)/urdf/open_manipulator.transmission.xacro" />
   <!-- World -->
   <link name="world">

File: urdf/right_open_manipulator.urdf.xacro (robot description, xacro)
@@ -7,5 +7,5 @@
   <xacro:include filename="$(find open_manipulator_description)/urdf/materials.xacro" />
   <!-- Import Transmission -->
-  <xacro:include filename="$(find open_manipulator_description)/urdf/transmission.xacro" />
+  <xacro:include filename="$(find open_manipulator_description)/urdf/open_manipulator.transmission.xacro" />
   <!-- World -->
   <link name="world">
@@ -13,5 +13,5 @@
   <!-- World fixed joint-->
   <joint name="world_fixed" type="fixed">
-    <origin xyz="0.1 0 0.5" rpy="0 -1.57079632679 0"/>
+    <origin xyz="0.1 0 0.5" rpy="0 1.57079632679 0"/>
     <parent link="world"/>
     <child link="link1"/>
